File: kicad/Timer2_timekeeping.kicad_pcb (KiCad board)
At the start: 2 copper layers, 45.5 x 57 mm, 15 parts, among them J1 Conn_01x02, SW1 SW_Push, SW2 SW_Push, SW3 SW_Push, SW4 SW_Push, U1 ATmega32A-P, Y1 Crystal

Commit message: small pcb update
Parts:
- removed BZ1: Buzzer, Buzzer_Beeper:Buzzer_12x9.5RM7.6
- added D2: LED, LED_THT:LED_D5.0mm, F.Cu at (145.0, 108.5)
- added D3: LED, LED_THT:LED_D5.0mm, F.Cu at (145.0, 116.0)
- added R3: 330, Resistor_THT:R_Axial_DIN0207_L6.3mm_D2.5mm_P7.62mm_Horizontal, F.Cu at (151.6, 106.8)
- added R4: 330, Resistor_THT:R_Axial_DIN0207_L6.3mm_D2.5mm_P7.62mm_Horizontal, F.Cu at (151.6, 110.8)
- moved J1 5.41 mm to (163.4, 108.9)
- moved D1 3.46 mm to (160.1, 101.4)
Connections:
- U1 pad 2: /ALARM_BUZZER -> /CPU_ACTIVE_LED
- U1 pad 3: unconnected-(U1-PB2-Pad3) -> /TIMER2_HEARTBEAT_LED
Routing:
- net /CPU_ACTIVE_LED: track 0.00 -> 61.2 mm
- net /TIMER2_HEARTBEAT_LED: track 0.00 -> 52.6 mm
- net /ALARM_BUZZER: track 51.9 -> 0.00 mm
- net GND: track 118.1 -> 168.8 mm
- net Net-(D3-K): track 0.00 -> 16.3 mm
- net Net-(D2-K): track 0.00 -> 15.8 mm
- net Net-(D1-K): track 15.5 -> 11.7 mm
- net Net-(J1-Pin_1): track 41.7 -> 41.1 mm
